Commit message: added sample code

File: urdf/arm_needle.urdf.xacro (robot description, xacro)
@@ -1,5 +1,5 @@
 <?xml version="1.0"?>
 <!-- Revolute-Revolute Manipulator -->
-<robot name="rrbot" xmlns:xacro="http://www.ros.org/wiki/xacro">
+<robot name="needle_bot" xmlns:xacro="http://www.ros.org/wiki/xacro">
   <xacro:include filename="$(find needle_simulation)/urdf/common_properties.xacro"/>
   <!-- Constants for robot dimensions -->

File: urdf/needle.urdf.xacro (robot description, xacro)
@@ -1,4 +1,4 @@
 <?xml version="1.0" ?>
-<robot name="aka_robot" xmlns:xacro="http://ros.org/wiki/xacro">
+<robot name="needle_bot" xmlns:xacro="http://ros.org/wiki/xacro">
   <xacro:include filename="$(find needle_simulation)/urdf/common_properties.xacro"/>
   <xacro:property name="base_width" value="0.1" /> <!-- Base -->
@@ -18,4 +18,19 @@
     </plugin>
   </gazebo>
+  <gazebo reference="base_link">
+    <material>Gazebo/Orange</material>
+  </gazebo>
+  <gazebo reference="upper_base_link">
+    <material>Gazebo/Black</material>
+  </gazebo>
+  <gazebo reference="prismatic_link">
+    <material>Gazebo/Yellow</material>
+  </gazebo>
+  <gazebo reference="motor_link">
+    <material>Gazebo/Orange</material>
+  </gazebo>
+  <gazebo reference="needle_link">
+    <material>Gazebo/Black</material>
+  </gazebo>
   <joint name="base_joint" type="fixed">
     <parent link="base_footprint"/>
@@ -69,8 +84,9 @@
     <inertial>
       <origin xyz="-${base_width/2} 0 0.0" rpy="0 1.57 0"/>
-      <mass value="8.2573504e-01"/>
-      <inertia ixx="2.2124416e-03" ixy="-1.2294101e-05" ixz="3.4938785e-05"
-               iyy="2.1193702e-03" iyz="-5.0120904e-06"
-               izz="2.0064271e-03" />
+      <mass value="${base_mass}"/>
+      <inertia
+	      ixx="${base_mass/ 12.0 * (base_width*base_width + base_length*base_length)}" ixy="0.0" ixz="0.0"
+	      iyy="${base_mass/ 12.0 * (base_length*base_length + base_width*base_width)}" iyz="0.0"
+	      izz="${base_mass/ 12.0 * (base_width*base_width + base_width*base_width)}"/>
     </inertial>
   </link>
@@ -79,12 +95,12 @@
     <child link="prismatic_link"/>
     <origin xyz="0 0 0" rpy="0 0 0"/>
-    <limit effort="30" velocity="0.5" lower="0" upper="${roto_linear_length}" />
+    <limit effort="30" velocity="0.1" lower="0" upper="${roto_linear_length}" />
     <axis xyz="1 0 0"/>
   </joint>
   <link name="prismatic_link">
     <visual>
-      <origin xyz="${motor_length/2} 0 -${(base_length/2)-(base_width/4)}" rpy="0 0 0"/>
-      <geometry>
-        <box size="${motor_length} ${motor_radius*2} ${base_width/2}"/>
+      <origin xyz="${motor_length/2} 0 -${(base_length/2)-((base_width*4/3)/2)}" rpy="0 0 0"/>
+      <geometry>
+        <box size="${motor_length*4/5} ${motor_radius*2} ${base_width*4/3}"/>
       </geometry>
       <material name="orange"/>
@@ -108,5 +124,5 @@
     <parent link="prismatic_link"/>
     <child link="motor_link"/>
-    <limit effort="30" velocity="1.57079633" lower="-1.57079633" upper="1.57079633" />
+    <limit effort="30" velocity="0.1" lower="-1.57079633" upper="1.57079633" />
     <origin xyz="0 0 0" rpy="0 0 0"/>
     <axis xyz="1 0 0"/>
