Commit message: added mpc and visualize the position on rviz

File: urdf/common_properties.xacro (robot description, xacro)
@@ -20,4 +20,7 @@
     <color rgba="0.5 0.5 0.5 1.0"/>
   </material>
+  <material name="yellow">
+    <color rgba="1.0 1.0 0.0 1.0"/>
+  </material>
   <material name="orange">
     <color rgba="${255/255} ${108/255} ${10/255} 1.0"/>

File: urdf/needle.urdf.xacro (robot description, xacro)
@@ -104,5 +104,5 @@
         <box size="${motor_length*4/5} ${motor_radius*2} ${base_width*4/3}"/>
       </geometry>
-      <material name="orange"/>
+      <material name="yellow"/>
     </visual>
     <!-- <collision>
